File: board/penta.kicad_pcb (KiCad board)
At the start: 4 copper layers, 37.4 x 37.4 mm, 186 parts, among them J1 USB_C_Receptacle, J2 USB_C_Receptacle, J3 Conn_01x03_Pin, Q1 Q_NMOS_SGD, SW1 SW_Push, U1 3.3V LDO, U2 RP2040, U3 QSPI Flash, U4 MSUSB30, U5 USBLC6-2P6, Y1 12MHz

Commit message: minor layout tweaks and drc
Routing:
- net Net-(J2-SHIELD): track 1.87 -> 13.2 mm, vias 0 -> 2
Changed lines of the file:
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@@
 		(sheetname "Root")
 		(sheetfile "penta.kicad_sch")
-		(attr smd)
+		(attr smd allow_soldermask_bridges)
 		(fp_circle
 			(center 0 -0.71)
@@
 		)
 		(fp_line
-			(start 1.325 -1.75)
-			(end 1.325 -0.035)
+			(start 1.325 -0.035)
+			(end 1.325 -1.75)
 			(stroke
 				(width 0.127)
@@
 		)
 		(fp_line
-			(start 0.45 -1.75)
-			(end 1.325 -1.75)
+			(start 1.325 -1.75)
+			(end 0.45 -1.75)
 			(stroke
 				(width 0.127)
@@
 		)
 		(fp_line
-			(start 0.16 1.75)
-			(end -0.16 1.75)
+			(start -0.16 1.75)
+			(end 0.16 1.75)
 			(stroke
 				(width 0.127)
@@
 		)
 		(fp_line
-			(start -1.325 -1.75)
-			(end -0.45 -1.75)
+			(start -0.45 -1.75)
+			(end -1.325 -1.75)
 			(stroke
 				(width 0.127)
@@
 		)
 		(fp_line
-			(start -1.325 -1.75)
-			(end -1.325 -0.035)
+			(start -1.325 -0.035)
+			(end -1.325 -1.75)
 			(stroke
 				(width 0.127)
@@
 		(fp_line
 			(start 1.575 2)
-			(end -1.575 2)
+			(end 1.575 -2)
 			(stroke
 				(width 0.05)
@@
 		(fp_line
 			(start 1.575 -2)
-			(end 1.575 2)
+			(end -1.575 -2)
 			(stroke
 				(width 0.05)
@@
 		(fp_line
 			(start -1.575 2)
-			(end -1.575 -2)
+			(end 1.575 2)
 			(stroke
 				(width 0.05)
@@
 		(fp_line
 			(start -1.575 -2)
-			(end 1.575 -2)
+			(end -1.575 2)
 			(stroke
 				(width 0.05)
@@
 		(fp_line
 			(start 1.325 1.75)
-			(end -1.325 1.75)
+			(end 1.325 -1.75)
 			(stroke
 				(width 0.127)
@@
 		(fp_line
 			(start 1.325 -1.75)
-			(end 1.325 1.75)
+			(end -1.325 -1.75)
 			(stroke
 				(width 0.127)
@@
 		(fp_line
 			(start -1.325 1.75)
-			(end -1.325 -1.75)
+			(end 1.325 1.75)
 			(stroke
 				(width 0.127)
@@
 		(fp_line
 			(start -1.325 -1.75)
-			(end 1.325 -1.75)
+			(end -1.325 1.75)
 			(stroke
 				(width 0.127)
@@
 	)
 	(via
-		(at 91.0082 106.9848)
+		(at 90.6272 107.061)
 		(size 0.6)
 		(drill 0.3)
@@
 	)
 	(segment
+		(start 92.742655 100.9142)
+		(end 92.774854 100.882001)
+		(width 0.4)
+		(layer "B.Cu")
+		(net 2)
+	)
+	(segment
 		(start 108.5964 102.4522)
 		(end 109.2454 101.8032)
@@
 	)
 	(segment
+		(start 91.5568 100.2182)
+		(end 91.975 100.6364)
+		(width 0.4)
+		(layer "B.Cu")
+		(net 2)
+	)
+	(segment
 		(start 90.0176 103.8606)
 		(end 89.789 104.0892)
@@
 	)
 	(segment
-		(start 91.8914 100.725)
-		(end 91.975 100.725)
-		(width 0.4)
-		(layer "B.Cu")
-		(net 2)
-	)
-	(segment
 		(start 106.8464 104.1796)
 		(end 106.491 104.1796)
@@
 	)
 	(segment
+		(start 91.975 100.6364)
+		(end 91.975 100.725)
+		(width 0.4)
+		(layer "B.Cu")
+		(net 2)
+	)
+	(segment
 		(start 107.3262 88.329)
 		(end 107.3262 89.094)
@@
 	)
 	(segment
+		(start 91.3846 100.2182)
+		(end 91.5568 100.2182)
+		(width 0.4)
+		(layer "B.Cu")
+		(net 2)
+	)
+	(segment
 		(start 103.770811 93.790389)
 		(end 103.9876 93.5736)
@@
 	)
 	(segment
+		(start 91.975 100.725)
+		(end 92.1642 100.9142)
+		(width 0.4)
+		(layer "B.Cu")
+		(net 2)
+	)
+	(segment
 		(start 96.266 94.4398)
 		(end 96.2914 94.4144)
@@
 	)
 	(segment
+		(start 92.1642 100.9142)
+		(end 92.742655 100.9142)
+		(width 0.4)
+		(layer "B.Cu")
+		(net 2)
+	)
+	(segment
 		(start 103.8606 89.824998)
 		(end 103.8606 88.4174)
@@
 	)
 	(segment
-		(start 107.0214 104.1796)
-		(end 108.4214 102.7796)
-		(width 0.2)
+		(start 90.6272 107.061)
+		(end 91.1352 107.061)
+		(width 0.15)
 		(layer "B.Cu")
 		(net 2)
 	)
 	(segment
-		(start 91.0082 106.9848)
-		(end 91.599008 106.393992)
-		(width 0.15)
+		(start 107.0214 104.1796)
+		(end 108.4214 102.7796)
+		(width 0.2)
 		(layer "B.Cu")
 		(net 2)
@@
 	)
 	(segment
-		(start 91.3846 100.2182)
-		(end 91.8914 100.725)
-		(width 0.4)
-		(layer "B.Cu")
-		(net 2)
-	)
-	(segment
 		(start 104.9528 109.0422)
 		(end 105.4608 108.5342)
@@
 	)
 	(segment
-		(start 91.599008 106.393992)
-		(end 91.8464 106.393992)
-		(width 0.15)
-		(layer "B.Cu")
-		(net 2)
-	)
-	(segment
 		(start 93.728 87.3232)
 		(end 93.8276 87.2236)
@@
 	)
 	(segment
+		(start 95.7072 85.0392)
+		(end 103.405448 85.0392)
+		(width 0.15)
+		(layer "F.Cu")
+		(net 145)
+	)
+	(segment
+		(start 103.405448 85.0392)
+		(end 103.583164 84.861484)
+		(width 0.15)
+		(layer "F.Cu")
+		(net 145)
+	)
+	(via
+		(at 103.583164 84.861484)
+		(size 0.6)
+		(drill 0.3)
+		(layers "F.Cu" "B.Cu")
+		(net 145)
+	)
+	(via
+		(at 95.7072 85.0392)
+		(size 0.6)
+		(drill 0.3)
+		(layers "F.Cu" "B.Cu")
+		(net 145)
+	)
+	(segment
+		(start 103.583164 84.861484)
+		(end 104.39728 85.6756)
+		(width 0.15)
+		(layer "B.Cu")
+		(net 145)
+	)
+	(segment
+		(start 94.670001 85.675599)
+		(end 95.070801 85.675599)
+		(width 0.15)
+		(layer "B.Cu")
+		(net 145)
+	)
+	(segment
+		(start 104.39728 85.6756)
+		(end 105.33 85.6756)
+		(width 0.15)
+		(layer "B.Cu")
+		(net 145)
+	)
+	(segment
+		(start 95.070801 85.675599)
+		(end 95.7072 85.0392)
+		(width 0.15)
+		(layer "B.Cu")
+		(net 145)
+	)
+	(segment
 		(start 105.33 85.6756)
 		(end 105.6928 85.6756)
@@
 	)
 	(via
-		(at 96.140963 108.409504)
+		(at 96.2406 108.5596)
 		(size 0.6)
 		(drill 0.3)
@@
 	)
 	(segment
+		(start 96.175801 108.5596)
+		(end 96.2406 108.5596)
+		(width 0.25)
+		(layer "B.Cu")
+		(net 184)
+	)
+	(segment
 		(start 97.8 103.939603)
 		(end 97.32468 104.414923)
@@
 	)
 	(segment
-		(start 96.140963 108.409504)
-		(end 96.140963 108.301637)
+		(start 96.1644 108.548199)
+		(end 96.175801 108.5596)
 		(width 0.25)
 		(layer "B.Cu")
@@
 	)
 	(segment
-		(start 97.8 103.4375)
-		(end 97.8 103.939603)
-		(width 0.2)
+		(start 96.1644 108.2782)
+		(end 96.1644 108.548199)
+		(width 0.25)
 		(layer "B.Cu")
 		(net 184)
 	)
 	(segment
-		(start 96.140963 108.301637)
-		(end 96.1644 108.2782)
-		(width 0.25)
+		(start 97.8 103.4375)
+		(end 97.8 103.939603)
+		(width 0.2)
 		(layer "B.Cu")
 		(net 184)
 	)
 	(segment
-		(start 96.140963 105.992237)
+		(start 97.32468 104.414923)
 		(end 97.32468 104.80852)
 		(width 0.2)
@@
 	(segment
 		(start 97.32468 104.80852)
-		(end 97.32468 104.414923)
+		(end 96.2406 105.8926)
 		(width 0.2)
 		(layer "In1.Cu")
@@
 	)
 	(segment
-		(start 96.140963 108.409504)
-		(end 96.140963 105.992237)
+		(start 96.2406 105.8926)
+		(end 96.2406 108.5596)
 		(width 0.2)
 		(layer "In1.Cu")
@@
 	)
 	(segment
+		(start 95.0976 107.823)
+		(end 95.0976 108.2274)
+		(width 0.2)
+		(layer "B.Cu")
+		(net 189)
+	)
+	(segment
 		(start 97.1971 103.4375)
 		(end 96.6724 103.9622)
@@
 	)
 	(segment
+		(start 95.0976 108.2274)
+		(end 95.1484 108.2782)
+		(width 0.2)
+		(layer "B.Cu")
+		(net 189)
+	)
+	(segment
 		(start 97.4 103.4375)
 		(end 97.1971 103.4375)
@@
 		(polygon
 			(pts
-				(xy 104.021228 105.534746) (xy 115.4938 105.0544) (xy 105.7656 97.9424)
+				(xy 104.021228 105.534746) (xy 115.4938 105.0544) (xy 105.7656 97.9678)
 			)
 		)
@@
 		(polygon
 			(pts
-				(xy 84.5312 104.9528) (xy 93.9292 97.9932) (xy 95.978771 105.534746)
+				(xy 84.5312 104.9528) (xy 93.9292 98.0186) (xy 95.9358 105.4862)
 			)
 		)
@@
 			)
 		)
+	)
+	(zone
+		(net 2)
+		(net_name "GND")
+		(layer "B.Cu")
+		(hatch edge 0.5)
+		(priority 6)
+		(connect_pads yes
+			(clearance 0.15)
+		)
+		(min_thickness 0.15)
+		(filled_areas_thickness no)
+		(fill yes
+			(thermal_gap 0.5)
+			(thermal_bridge_width 0.5)
+			(island_removal_mode 1)
+			(island_area_min 10)
+		)
+		(polygon
+			(pts
+				(xy 90.4748 106.9594) (xy 91.186 106.5784) (xy 91.186 107.5182) (xy 90.4748 107.1626) (xy 90.4748 106.934)
+			)
+		)

Commit message: mosfet GSD was actually correct so change it back. the dim pixel issue was current leaking through data line, already fixed in software in main
Parts:
- Q1: value Q_NMOS_SGD -> Q_NMOS_GSD
- turned D108 to -53.181 degrees
- turned D113 to -85.909 degrees
- turned D87 to 84.272 degrees
- turned R12 to -90 degrees
Connections:
- Q1 pad 1: GND -> /EN_PIXELS
- Q1 pad 2: /EN_PIXELS -> GND
Routing:
- net GND: track 54.9 -> 52.6 mm, vias 53 -> 51
